Commit message: Attached the lidar to the myrobo and try it

File: urdf/robo_core.xacro (robot description, xacro)
@@ -13,3 +13,6 @@
         <color rgba="0 0 0 1"/>
     </material>
+    <material name="red">
+        <color rgba="1 0 0 0"/>
+    </material>
 </robot>

File: urdf/robot1.xacro (robot description, xacro)
@@ -19,7 +19,7 @@
   <xacro:property name="joint_right_wheel_y" value="${(chassis_size_y/2)+(wheel_length/2)}" />
   <!-- <xacro:property name="joint_right_wheel_z" value="0" /> -->
-  <xacro:property name="lidar_x" value="0" />
-  <xacro:property name="lidar_y" value="${-1*chassis_size_y/2}" />
-  <xacro:property name="lidar_z" value="${wheel_radius+chassis_size_z}" />
+  <xacro:property name="lidar_x" value="0.1" />
+  <xacro:property name="lidar_y" value="0" />
+  <xacro:property name="lidar_z" value="0.175" />
   <xacro:property name="lidar_z_offset" value="0" />
   <xacro:property name="chassis_mass" value="0.7" />
@@ -57,5 +57,5 @@
   </link>
   <gazebo reference = "chassis">
-      <material>Gazebo/White</material>
+      <material>Gazebo/Red</material>
   </gazebo>
    <!-- righ wheel-->
@@ -134,5 +134,5 @@
   </link>
   <gazebo reference = "caster_link">
-    <material>Gazebo/Black</material>
+    <material>Gazebo/Silver</material>
     <!-- gazebo adding the coeffecient of friction -->
     <mu1 value="0.001" />
@@ -140,7 +140,6 @@
   </gazebo>
   <!-- lidar -->
-<!--
   <joint name="lidar_joint" type="fixed">
-    <origin xyz="${lidar_x} ${lidar_y} ${lidar_z}" rpy="0 0 -1.5708"/>
+    <origin xyz="${lidar_x} ${lidar_y} ${lidar_z}" rpy="0 0 0"/>
     <parent link="chassis"/>
     <child link="lidar"/>
@@ -164,4 +163,7 @@
       <inertia ixx="1e-6" ixy="0" ixz="0" iyy="1e-6" iyz="0" izz="1e-6" />
     </inertial>
-  </link> -->
+  </link>
+  <gazebo reference = "lidar">
+    <material>Gazebo/Black</material>
+  </gazebo>
 </robot>
