Commit message: Editing URDF

File: urdf/robot1.xacro (robot description, xacro)
@@ -1,19 +1,22 @@
 <?xml version="1.0" encoding="UTF-8"?>
-<robot xmlns:xacro="http://www.ros.org/wiki/xacro" name="robot1">
+<robot xmlns:xacro="http://www.ros.org/wiki/xacro"  name="robot1" >
+  <xacro:include filename="robo_core.xacro" />
+  <xacro:include filename="inertial.xacro" />
   <xacro:include filename="$(find test)/urdf/plugin.gazebo" />
-  <xacro:property name="chassis_x" value="0" />
-  <xacro:property name="chassis_y" value="0" />
-  <xacro:property name="chassis_z" value="0" />
-  <xacro:property name="chassis_offset_z" value="${wheel_radius+chassis_size_z/2}" />
-  <xacro:property name="chassis_size_x" value="0.5" />
-  <xacro:property name="chassis_size_y" value="0.7" />
-  <xacro:property name="chassis_size_z" value="0.1" />
-  <xacro:property name="wheel_radius" value="0.15" />
-  <xacro:property name="wheel_length" value="0.09" />
+  <!-- behind the center of the two drive wheels to make the robot accelerated easier  -->
+  <xacro:property name="chassis_x" value="-0.1" />
+  <!-- <xacro:property name="chassis_y" value="0" />
+  <xacro:property name="chassis_z" value="0" /> -->
+  <xacro:property name="chassis_offset_z" value="${chassis_size_z/2}" />
+  <xacro:property name="chassis_offset_x" value="${chassis_size_x/2}" />
+  <xacro:property name="chassis_size_x" value="0.3" />
+  <xacro:property name="chassis_size_y" value="0.3" />
+  <xacro:property name="chassis_size_z" value="0.15" />
+  <xacro:property name="wheel_radius" value="0.05" />
+  <xacro:property name="wheel_length" value="0.04" />
 -
-  <xacro:property name="joint_right_wheel_x" value="0.25" />
-  <xacro:property name="joint_right_wheel_y" value="0.175" />
-  <xacro:property name="joint_right_wheel_z" value="0.1" />
-  <xacro:property name="right_wheel_offset" value="${wheel_length/2}" />
+  <!-- <xacro:property name="joint_right_wheel_x" value="0" /> -->
+  <xacro:property name="joint_right_wheel_y" value="${(chassis_size_y/2)+(wheel_length/2)}" />
+  <!-- <xacro:property name="joint_right_wheel_z" value="0" /> -->
   <xacro:property name="lidar_x" value="0" />
   <xacro:property name="lidar_y" value="${-1*chassis_size_y/2}" />
@@ -23,126 +26,119 @@
   <xacro:property name="wheel_mass" value="0.1" />
   <xacro:property name="caster_mass" value="0.05" />
-  <link name="base_footprint">
+  <xacro:property name="caster_x" value="0.24" />
+  <xacro:property name="caster_radius" value="0.05" />
+  <xacro:property name="CW" value="-1" />
+  <xacro:property name="CCW" value="1" />
+  <link name="base_link">
   </link>
   <!-- Chassis-->
 <joint name="chassis_joint" type="fixed">
-  <origin xyz="${chassis_x} ${chassis_y} ${chassis_z}" rpy="0.0 0.0 0.0"/>
-  <parent link="base_footprint"/>
+  <origin xyz="${chassis_x} 0 0" />
+  <parent link="base_link"/>
   <child link="chassis"/>
 </joint>
   <link name="chassis">
-    <inertial>
-      <origin xyz="0.0 0.0 ${chassis_offset_z}" rpy="0.0 0.0 0.0"/>
-      <mass value="${chassis_mass}"/>
-      <inertia ixx="0.1" ixy="0.0" ixz="0.0" iyy="0.1" iyz="0.0" izz="0.1"/>
-    </inertial>
     <visual name="">
-      <origin xyz="0.0 0.0 ${chassis_offset_z}" rpy="0.0 0.0 0.0"/>
+      <origin xyz="${chassis_offset_x} 0 ${chassis_offset_z}" />
       <geometry>
         <box size="${chassis_size_x} ${chassis_size_y} ${chassis_size_z}"/>
       </geometry>
-      <material name="">
-        <color rgba="1.0 1.0 1.0 1.0"/>
-        <texture filename=""/>
-      </material>
+      <material name="white"/>
     </visual>
-    <collision>
-      <origin xyz="0.0 0.0 ${chassis_offset_z}" rpy="0.0 0.0 0.0"/>
+    <collision name="">
+      <origin xyz="${chassis_offset_x} 0 ${chassis_offset_z}" />
       <geometry>
         <box size="${chassis_size_x} ${chassis_size_y} ${chassis_size_z}"/>
       </geometry>
     </collision>
+    <xacro:inertial_box mass="0.5" x="${chassis_size_x}" y="${chassis_size_y}" z="${chassis_size_z}">
+      <origin xyz="${chassis_offset_x} 0 ${chassis_offset_z}" rpy ="0 0 0"/>
+    </xacro:inertial_box>
   </link>
+  <gazebo reference = "chassis">
+      <material>Gazebo/White</material>
+  </gazebo>
    <!-- righ wheel-->
-  <joint name="right_wheel_joint" type="continuous">
-    <origin xyz="${joint_right_wheel_x} ${joint_right_wheel_y} ${wheel_radius}" rpy="0.0 1.5708 0.0"/>
-    <parent link="chassis"/>
+   <joint name="right_wheel_joint" type="continuous">
+    <origin xyz="0 -${joint_right_wheel_y} 0" rpy="${CCW*(pi/2)} 0 0.0"/>
+    <parent link="base_link"/>
     <child link="right_wheel"/>
-    <axis xyz="0 0.0 -1"/>
+    <axis xyz="0 0.0 ${CW}"/>
   </joint>
   <link name="right_wheel">
-    <inertial>
-      <origin xyz="0 0.0 ${right_wheel_offset}" rpy="0.0 0.0 0.0"/>
-      <mass value="${wheel_mass}"/>
-      <inertia ixx="0.1" ixy="0.0" ixz="0.0" iyy="0.1" iyz="0.0" izz="0.1"/>
-    </inertial>
     <visual name="">
-      <origin xyz="0 0.0 ${right_wheel_offset}" rpy="0.0 0.0 0.0"/>
       <geometry>
         <cylinder radius="${wheel_radius}" length="${wheel_length}"/>
       </geometry>
-      <material name="">
-        <color rgba="0.2 1.0 0.2 1.0"/>
-        <texture filename=""/>
-      </material>
+      <material name="blue"/>
     </visual>
-    <collision>
-      <origin xyz="0 0.0 ${right_wheel_offset}" rpy="0.0 0.0 0.0"/>
+    <collision name="">
       <geometry>
         <cylinder radius="${wheel_radius}" length="${wheel_length}"/>
       </geometry>
     </collision>
-  </link>
+    <xacro:inertial_cylinder mass="0.1" length="${wheel_length}" radius="${wheel_radius}">
+        <origin xyz="0 0 0" rpy="0 0 0"/>
+    </xacro:inertial_cylinder>
+  </link> -->
+  <gazebo reference = "right_wheel">
+    <material>Gazebo/Blue</material>
+  </gazebo>
   <!-- left wheel-->
   <joint name="left_wheel_joint" type="continuous">
-    <origin xyz="${-1*joint_right_wheel_x} ${joint_right_wheel_y} ${wheel_radius}" rpy="0.0 -1.5708 0.0"/>
-    <parent link="chassis"/>
+    <origin xyz="0 ${joint_right_wheel_y} 0" rpy="${CW*(pi/2)} 0 0.0"/>
+    <parent link="base_link"/>
     <child link="left_wheel"/>
-    <axis xyz="0 0.0 -1"/>
+    <axis xyz="0 0 ${CCW}"/>
   </joint>
   <link name="left_wheel">
-    <inertial>
-      <origin xyz="0 0.0 ${right_wheel_offset}" rpy="0.0 0.0 0.0"/>
-      <mass value="${wheel_mass}"/>
-      <inertia ixx="0.1" ixy="0.0" ixz="0.0" iyy="0.1" iyz="0.0" izz="0.1"/>
-    </inertial>
     <visual name="">
-      <origin xyz="0 0.0 ${right_wheel_offset}" rpy="0.0 0.0 0.0"/>
       <geometry>
         <cylinder radius="${wheel_radius}" length="${wheel_length}"/>
       </geometry>
-      <material name="">
-        <color rgba="0.2 1.0 0.2 1.0"/>
-        <texture filename=""/>
-      </material>
+      <material name="blue"/>
     </visual>
-    <collision>
-      <origin xyz="0 0.0 ${right_wheel_offset}" rpy="0.0 0.0 0.0"/>
+    <collision name="">
       <geometry>
         <cylinder radius="${wheel_radius}" length="${wheel_length}"/>
       </geometry>
     </collision>
-  </link>
+    <xacro:inertial_cylinder mass="0.1" length="${wheel_length}" radius="${wheel_radius}">
+      <origin xyz="0 0 0" rpy="0 0 0"/>
+    </xacro:inertial_cylinder>
+  </link> -->
+  <gazebo reference = "left_wheel">
+    <material>Gazebo/Blue</material>
+  </gazebo>
   <!-- caster wheel-->
-  <joint name="caster_joint" type="continuous">
-    <origin xyz="0 -0.25 ${wheel_radius/2}" rpy="0.0 -1.5708 0.0"/>
+  <joint name="caster_joint" type="fixed">
+    <origin xyz="${caster_x} 0 0" />
     <parent link="chassis"/>
     <child link="caster_link"/>
-    <axis xyz="0.0 0.0 1.0"/>
   </joint>
   <link name="caster_link">
-    <inertial>
-        <origin xyz="0.0 0.0 0.0" rpy="0.0 0.0 0.0"/>
-        <mass value="${caster_mass}"/>
-        <inertia ixx="0.1" ixy="0.0" ixz="0.0" iyy="0.1" iyz="0.0" izz="0.1"/>
-    </inertial>
     <visual name="">
-        <origin xyz="0.0 0.0 0.0" rpy="0.0 0.0 0.0"/>
         <geometry>
-            <cylinder radius="${wheel_radius/2}" length="${wheel_length}"/>
+            <sphere radius="${caster_radius}"/>
         </geometry>
-        <material name="">
-            <color rgba="1.0 0.0 0.0 1.0"/>
-            <texture filename=""/>
-        </material>
+        <material name="black"/>
     </visual>
-    <collision>
-        <origin xyz="0.0 0.0 0.0" rpy="0.0 0.0 0.0"/>
-        <geometry>
-            <cylinder radius="${wheel_radius/2}" length="${wheel_length}"/>
-        </geometry>
+    <collision name="">
+      <geometry>
+          <sphere radius="${caster_radius}"/>
+      </geometry>
     </collision>
+    <xacro:inertial_sphere mass="0.1" radius="${wheel_radius}">
+      <origin xyz="0 0 0" rpy="0 0 0"/>
+    </xacro:inertial_sphere>
   </link>
+  <gazebo reference = "caster_link">
+    <material>Gazebo/Black</material>
+    <!-- gazebo adding the coeffecient of friction -->
+    <mu1 value="0.001" />
+    <mu2 value="0.001" />
+  </gazebo>
   <!-- lidar -->
+<!--
   <joint name="lidar_joint" type="fixed">
     <origin xyz="${lidar_x} ${lidar_y} ${lidar_z}" rpy="0 0 -1.5708"/>
@@ -168,4 +164,4 @@
       <inertia ixx="1e-6" ixy="0" ixz="0" iyy="1e-6" iyz="0" izz="1e-6" />
     </inertial>
-  </link>
+  </link> -->
 </robot>

Commit message: adding code and readme

File: urdf/robot1.xacro (robot description, xacro)
@@ -19,5 +19,5 @@
   <xacro:property name="joint_right_wheel_y" value="${(chassis_size_y/2)+(wheel_length/2)}" />
   <!-- <xacro:property name="joint_right_wheel_z" value="0" /> -->
-  <xacro:property name="lidar_x" value="0.1" />
+  <xacro:property name="lidar_x" value="0.275" />
   <xacro:property name="lidar_y" value="0" />
   <xacro:property name="lidar_z" value="0.175" />

Commit message: Editing Project Name and MD Files

File: urdf/robot1.xacro (robot description, xacro)
@@ -3,5 +3,5 @@
   <xacro:include filename="robo_core.xacro" />
   <xacro:include filename="inertial.xacro" />
-  <xacro:include filename="$(find test)/urdf/plugin.gazebo" />
+  <xacro:include filename="$(find Differential-Drive-Robot-using-ROS)/urdf/plugin.gazebo" />
   <!-- behind the center of the two drive wheels to make the robot accelerated easier  -->
   <xacro:property name="chassis_x" value="-0.1" />
@@ -149,5 +149,5 @@
       <origin xyz="0 0 ${lidar_z_offset}" rpy="0 0 0"/>
       <geometry>
-        <mesh filename="package://test/meshes/hokuyo.dae"/>
+        <mesh filename="package://Differential-Drive-Robot-using-ROS/meshes/hokuyo.dae"/>
       </geometry>
     </collision>
@@ -155,5 +155,5 @@
         <origin xyz="0 0 ${lidar_z_offset}" rpy="0 0 0"/>
         <geometry>
-        <mesh filename="package://test/meshes/hokuyo.dae"/>
+        <mesh filename="package://Differential-Drive-Robot-using-ROS/meshes/hokuyo.dae"/>
       </geometry>
     </visual>
