Commit message: Editing urdf, gazebo, pkg name and md file

File: urdf/myrobo.xacro (robot description, xacro)
@@ -1,7 +1,7 @@
 <?xml version="1.0" encoding="UTF-8"?>
 <robot xmlns:xacro="http://www.ros.org/wiki/xacro"  name="robot1" >
-  <xacro:include filename="robo_core.xacro" />
+  <xacro:include filename="colour.xacro" />
   <xacro:include filename="inertial.xacro" />
-  <xacro:include filename="$(find Differential-Drive-Robot-using-ROS)/urdf/plugin.gazebo" />
+  <xacro:include filename="$(find myrobo_description)/urdf/plugin.gazebo" />
   <!-- behind the center of the two drive wheels to make the robot accelerated easier  -->
   <xacro:property name="chassis_x" value="-0.1" />
@@ -56,7 +56,4 @@
     </xacro:inertial_box>
   </link>
-  <gazebo reference = "chassis">
-      <material>Gazebo/Red</material>
-  </gazebo>
    <!-- righ wheel-->
    <joint name="right_wheel_joint" type="continuous">
@@ -82,7 +79,4 @@
     </xacro:inertial_cylinder>
   </link> -->
-  <gazebo reference = "right_wheel">
-    <material>Gazebo/Blue</material>
-  </gazebo>
   <!-- left wheel-->
   <joint name="left_wheel_joint" type="continuous">
@@ -108,7 +102,4 @@
     </xacro:inertial_cylinder>
   </link> -->
-  <gazebo reference = "left_wheel">
-    <material>Gazebo/Blue</material>
-  </gazebo>
   <!-- caster wheel-->
   <joint name="caster_joint" type="fixed">
@@ -133,10 +124,4 @@
     </xacro:inertial_sphere>
   </link>
-  <gazebo reference = "caster_link">
-    <material>Gazebo/Silver</material>
-    <!-- gazebo adding the coeffecient of friction -->
-    <mu1 value="0.001" />
-    <mu2 value="0.001" />
-  </gazebo>
   <!-- lidar -->
   <joint name="lidar_joint" type="fixed">
@@ -149,5 +134,5 @@
       <origin xyz="0 0 ${lidar_z_offset}" rpy="0 0 0"/>
       <geometry>
-        <mesh filename="package://Differential-Drive-Robot-using-ROS/meshes/hokuyo.dae"/>
+        <mesh filename="package://myrobo_description/meshes/hokuyo.dae"/>
       </geometry>
     </collision>
@@ -155,5 +140,5 @@
         <origin xyz="0 0 ${lidar_z_offset}" rpy="0 0 0"/>
         <geometry>
-        <mesh filename="package://Differential-Drive-Robot-using-ROS/meshes/hokuyo.dae"/>
+        <mesh filename="package://myrobo_description/meshes/hokuyo.dae"/>
       </geometry>
     </visual>
@@ -164,6 +149,3 @@
     </inertial>
   </link>
-  <gazebo reference = "lidar">
-    <material>Gazebo/Black</material>
-  </gazebo>
 </robot>
